File: hardware/motherboard-201/motherboard-201.kicad_pcb (KiCad board)
At the start: 2 copper layers, 216 x 150 mm, 106 parts, among them J1 PWR_conn, J2 PS2_CONN, J3 MSX_Slot, J4 MSX_Slot, J5 GFX_Connector_Output, J6 CONN_JOY, J7 CONN_JOY, J8 DIN8, K1 Relay, Q2 2N2907, U1 AS6C1008, U10 74HC670, U11 74HC670, U12 74HC670, U13 ATMEGA328P, U15 74HC139, U16 74LS07, U17 74HC74, U19 LM311, U2 TL7705, U20 SST39SF0, U23 74HC157, U24 AY-3-8910, U25 74HC157, U26 74HC138, U27 74HC153, U28 82C55A, U3 GAL_declogic-201, U4 74HC670, U5 74HC670, U6 Z84C00, U7 74HC74, U8 74HCT245, U9 74HC670, Y1 16Mhz

Commit message: [mb201] Set JLCPCB PCB capabilities
Other:
- net class Default: clearance 0.2032 -> 0.127; trace_width 0.2032 -> 0.127; via_dia 0.6 -> 0.5; via_drill 0.3 -> 0.25
- rule trace_clearance: 0.2032 -> 0.127
- rule trace_min: 0.1524 -> 0.127
- rule via_min_drill: 0.3 -> 0.2
- rule via_min_size: 0.6 -> 0.45
Changed lines of the file:
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@@
   )
   (setup
-    (last_trace_width 0.2032)
-    (trace_clearance 0.2032)
+    (last_trace_width 0.127)
+    (trace_clearance 0.127)
     (zone_clearance 0.2032)
     (zone_45_only no)
-    (trace_min 0.1524)
-    (via_size 0.6)
-    (via_drill 0.3)
-    (via_min_size 0.6)
-    (via_min_drill 0.3)
-    (uvia_size 0.6)
-    (uvia_drill 0.3)
-    (uvias_allowed no)
-    (uvia_min_size 0.6)
-    (uvia_min_drill 0.3)
+    (trace_min 0.127)
+    (via_size 0.5)
+    (via_drill 0.25)
+    (via_min_size 0.45)
+    (via_min_drill 0.2)
+    (uvia_size 0.5)
+    (uvia_drill 0.25)
+    (uvias_allowed yes)
+    (uvia_min_size 0.45)
+    (uvia_min_drill 0.2)
     (edge_width 0.15)
     (segment_width 0.2)
@@
   (net 214 "Net-(U15-Pad9)")
   (net_class Default "Esta es la clase de red por defecto."
-    (clearance 0.2032)
-    (trace_width 0.2032)
-    (via_dia 0.6)
-    (via_drill 0.3)
-    (uvia_dia 0.6)
-    (uvia_drill 0.3)
+    (clearance 0.127)
+    (trace_width 0.127)
+    (via_dia 0.5)
+    (via_drill 0.25)
+    (uvia_dia 0.5)
+    (uvia_drill 0.25)
     (diff_pair_width 0.1524)
     (diff_pair_gap 0.1524)
@@
     (add_net ~)
   )
+  (module artemisa:PS2_conn (layer F.Cu)
+    (at 272.796 130.81 90)
+    (clearance 0.1)
+    (fp_text reference J2 (at 0 -14 270) (layer F.SilkS)
+      (effects (font (size 1 1) (thickness 0.15)))
+    )
+    (fp_text value PS2_CONN (at -0.009088 0.88875 270) (layer F.Fab)
+      (effects (font (size 1 1) (thickness 0.15)))
+    )
+    (fp_line (start -7 -13) (end -8 -13) (layer F.SilkS) (width 0.15))
+    (fp_line (start -8 -13) (end -8 0) (layer F.SilkS) (width 0.15))
+    (fp_line (start -8 0) (end -7 0) (layer F.SilkS) (width 0.15))
+    (fp_line (start -7 -13) (end 7 -13) (layer F.SilkS) (width 0.15))
+    (fp_line (start 7 -13) (end 8 -13) (layer F.SilkS) (width 0.15))
+    (fp_line (start 8 -13) (end 8 0) (layer F.SilkS) (width 0.15))
+    (fp_line (start 8 0) (end 7 0) (layer F.SilkS) (width 0.15))
+    (fp_line (start -7 0) (end 3.4 0) (layer F.SilkS) (width 0.15))
+    (fp_line (start 3.4 0) (end 7 0) (layer F.SilkS) (width 0.15))
+    (pad "" thru_hole rect (at 6.85 -5.5) (size 3.5 1.5) (drill oval 3 1) (layers *.Cu *.Mask))
+    (pad "" thru_hole rect (at -6.85 -5.5) (size 3.5 1.5) (drill oval 3 1) (layers *.Cu *.Mask))
+    (pad "" thru_hole rect (at 0 -4.85 270) (size 3.5 1.5) (drill oval 3 1) (layers *.Cu *.Mask))
+    (pad 6 thru_hole circle (at -3.25 -11.3 270) (size 1.5 1.5) (drill 0.9) (layers *.Cu *.Mask)
+      (net 194 "Net-(J2-Pad6)"))
+    (pad 5 thru_hole circle (at 3.25 -11.3 270) (size 1.5 1.5) (drill 0.9) (layers *.Cu *.Mask)
+      (net 195 "Net-(J2-Pad5)"))
+    (pad 3 thru_hole circle (at 3.25 -8.5 270) (size 1.5 1.5) (drill 0.9) (layers *.Cu *.Mask)
+      (net 1 GND) (clearance 0.1))
+    (pad 4 thru_hole circle (at -3.25 -8.5 270) (size 1.5 1.5) (drill 0.9) (layers *.Cu *.Mask)
+      (net 119 ~) (clearance 0.1))
+    (pad 1 thru_hole circle (at 1.5 -8.5 270) (size 1.5 1.5) (drill 0.9) (layers *.Cu *.Mask)
+      (net 196 "Net-(J2-Pad1)"))
+    (pad 2 thru_hole circle (at -1.5 -8.5 270) (size 1.5 1.5) (drill 0.9) (layers *.Cu *.Mask)
+      (net 197 "Net-(J2-Pad2)"))
+    (model ${KIPRJMOD}/../libs/artemisa.3dshapes/PS2_conn.wrl
+      (offset (xyz 0 7.111999893188477 0))
+      (scale (xyz 1.025 1.1 1.1))
+      (rotate (xyz 0 0 0))
+    )
+  )
   (module artemisa:Crystal (layer F.Cu)
     (at 267.716 162.56 90)
@@
     )
   )
-  (module artemisa:PS2_conn (layer F.Cu)
-    (at 272.796 130.81 90)
-    (fp_text reference J2 (at 0 -14 270) (layer F.SilkS)
-      (effects (font (size 1 1) (thickness 0.15)))
-    )
-    (fp_text value PS2_CONN (at -0.009088 0.88875 270) (layer F.Fab)
-      (effects (font (size 1 1) (thickness 0.15)))
-    )
-    (fp_line (start -7 -13) (end -8 -13) (layer F.SilkS) (width 0.15))
-    (fp_line (start -8 -13) (end -8 0) (layer F.SilkS) (width 0.15))
-    (fp_line (start -8 0) (end -7 0) (layer F.SilkS) (width 0.15))
-    (fp_line (start -7 -13) (end 7 -13) (layer F.SilkS) (width 0.15))
-    (fp_line (start 7 -13) (end 8 -13) (layer F.SilkS) (width 0.15))
-    (fp_line (start 8 -13) (end 8 0) (layer F.SilkS) (width 0.15))
-    (fp_line (start 8 0) (end 7 0) (layer F.SilkS) (width 0.15))
-    (fp_line (start -7 0) (end 3.4 0) (layer F.SilkS) (width 0.15))
-    (fp_line (start 3.4 0) (end 7 0) (layer F.SilkS) (width 0.15))
-    (pad "" thru_hole rect (at 6.85 -5.5) (size 3.5 1.5) (drill oval 3 1) (layers *.Cu *.Mask))
-    (pad "" thru_hole rect (at -6.85 -5.5) (size 3.5 1.5) (drill oval 3 1) (layers *.Cu *.Mask))
-    (pad "" thru_hole rect (at 0 -4.85 270) (size 3.5 1.5) (drill oval 3 1) (layers *.Cu *.Mask))
-    (pad 6 thru_hole circle (at -3.25 -11.3 270) (size 1.5 1.5) (drill 0.9) (layers *.Cu *.Mask)
-      (net 194 "Net-(J2-Pad6)"))
-    (pad 5 thru_hole circle (at 3.25 -11.3 270) (size 1.5 1.5) (drill 0.9) (layers *.Cu *.Mask)
-      (net 195 "Net-(J2-Pad5)"))
-    (pad 3 thru_hole circle (at 3.25 -8.5 270) (size 1.5 1.5) (drill 0.9) (layers *.Cu *.Mask)
-      (net 1 GND))
-    (pad 4 thru_hole circle (at -3.25 -8.5 270) (size 1.5 1.5) (drill 0.9) (layers *.Cu *.Mask)
-      (net 119 ~))
-    (pad 1 thru_hole circle (at 1.5 -8.5 270) (size 1.5 1.5) (drill 0.9) (layers *.Cu *.Mask)
-      (net 196 "Net-(J2-Pad1)"))
-    (pad 2 thru_hole circle (at -1.5 -8.5 270) (size 1.5 1.5) (drill 0.9) (layers *.Cu *.Mask)
-      (net 197 "Net-(J2-Pad2)"))
-    (model ${KIPRJMOD}/../libs/artemisa.3dshapes/PS2_conn.wrl
-      (offset (xyz 0 7.111999893188477 0))
-      (scale (xyz 1.025 1.1 1.1))
-      (rotate (xyz 0 0 0))
-    )
-  )
   (module artemisa:C_1206 (layer F.Cu)
     (at 263.906 166.5 90)
@@
     (at 147.896 94.6)
     (descr "TO92 flat pins")
-    (clearance 0.15)
+    (clearance 0.1)
     (fp_text reference Q2 (at 3.81 -0.635) (layer F.SilkS)
       (effects (font (size 1 1) (thickness 0.15)))
